File: GL516_Template.kicad_pcb (KiCad board)
At the start: 2 copper layers, 314.4 x 98.8 mm, 90 parts, among them J10 Conn_01x01, J11 Conn_01x01, J12 Conn_01x01, J13 Conn_01x01, J14 Conn_01x01, J15 Conn_01x01, J16 Conn_01x01, J17 Conn_01x01, J2 Conn_01x01, J3 Conn_01x01, J4 Conn_01x01, J5 Conn_01x01, J6 Conn_01x01, J7 Conn_01x01, J8 Conn_01x01, J9 Conn_01x01, SW1 SW_PUSH, SW2 KEY_SWITCH, SW3 SW_PUSH, SW4 KEY_SWITCH, SW4 SW_PUSH, SW5 SW_PUSH, SW7 SW_PUSH, SW8 SW_PUSH

Commit message: テンプレートのスイッチリファレンスを変更
Parts:
- removed the SW8 at (257.2, 85.7)
- SW4: footprint kbd_SW_Hole:SW_Hole_2 -> kbd_SW_Hole:SW_Hole_2.25
- SW62: renamed from SW8; footprint kbd_SW_Hole:SW_Hole_1 -> kbd_SW_Hole:SW_Hole_1.75
- moved SW62 7.14 mm to (269.1, 85.7)
- moved SW39 4.76 mm to (185.7, 85.7)
- moved SW49 4.76 mm to (223.8, 85.7)
- moved SW14 4.76 mm to (90.5, 85.7)
- moved SW24 4.76 mm to (128.6, 85.7)
- moved SW9 4.76 mm to (71.4, 85.7)
- moved SW19 4.76 mm to (109.5, 85.7)
- moved SW29 4.76 mm to (147.6, 85.7)
- moved SW34 4.76 mm to (166.7, 85.7)
- moved SW44 4.76 mm to (204.8, 85.7)
- moved SW54 4.76 mm to (242.9, 85.7)
- moved SW4 2.38 mm to (40.5, 85.7)
- renumbered SW7 to SW10, SW4 to SW11, SW8 to SW12, SW4 to SW13, SW8 to SW14, SW7 to SW15, SW4 to SW16, SW8 to SW17, SW4 to SW18, SW8 to SW19, SW8 to SW20, SW4 to SW21, SW8 to SW22, SW4 to SW23, SW8 to SW24, SW5 to SW25, SW4 to SW26, SW8 to SW27, SW4 to SW28, SW8 to SW29, SW8 to SW30, SW4 to SW31, SW8 to SW32, SW4 to SW33, SW8 to SW34, SW8 to SW35, SW4 to SW36, SW8 to SW37, SW4 to SW38, SW8 to SW39, SW5 to SW40, SW4 to SW41, SW8 to SW42, SW4 to SW43, SW8 to SW44, SW8 to SW45, SW4 to SW46, SW8 to SW47, SW4 to SW48, SW8 to SW49, SW7 to SW5, SW5 to SW50, SW4 to SW51, SW8 to SW52, SW4 to SW53, SW8 to SW54, SW5 to SW55, SW4 to SW56, SW8 to SW57, SW4 to SW58, SW4 to SW59, SW4 to SW6, SW8 to SW60, SW4 to SW61, SW8 to SW63, SW4 to SW64, SW4 to SW65, SW4 to SW66, SW8 to SW67, SW8 to SW68, SW4 to SW69, SW8 to SW7, SW8 to SW70, SW4 to SW71, SW8 to SW72, SW8 to SW73, SW4 to SW8, SW8 to SW9

Commit message: フットプリント名の変更に対応
Parts:
- SW1, SW10, SW11, SW12, SW13, SW14, SW16, SW17, SW18, SW19, SW20, SW21, SW22, SW23, SW24, SW26, SW27, SW28, SW29, SW30, SW31, SW32, SW33, SW34, SW35, SW36, SW37, SW38, SW39, SW41, SW42, SW43, SW44, SW45, SW46, SW47, SW48, SW49, SW51, SW52, SW53, SW54, SW56, SW57, SW58, SW59, SW6, SW60, SW61, SW63, SW64, SW65, SW67, SW68, SW69, SW7, SW70, SW71, SW72, SW73, SW8, SW9: footprint kbd_SW_Hole:SW_Hole_1 -> kbd_SW_Hole:SW_Hole_1u
- SW15, SW25, SW40, SW5, SW50, SW55: footprint kbd_SW_Hole:SW_Hole_1.25 -> kbd_SW_Hole:SW_Hole_1.25u
- SW2: footprint kbd_SW_Hole:SW_Hole_1.5 -> kbd_SW_Hole:SW_Hole_1.5u
- SW3, SW62: footprint kbd_SW_Hole:SW_Hole_1.75 -> kbd_SW_Hole:SW_Hole_1.75u
- SW4: footprint kbd_SW_Hole:SW_Hole_2.25 -> kbd_SW_Hole:SW_Hole_2.25u
- SW66: footprint kbd_SW_Hole:SW_Hole_2 -> kbd_SW_Hole:SW_Hole_2u
